File: TL431_VoltageSupply.sch (EAGLE design)
At the start: 12 parts, among them P1 LSP10, P2 LSP10, P3 LSP10, P4 LSP10, T1 BD139

Commit message: Add files via upload
Other:
- note added: "https://github.com/pksato/TL431-Circuits"
Changed lines of the file:
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@@
 <setting verticaltext="up"/>
 </settings>
-<grid distance="0.1" unitdist="inch" unit="inch" style="lines" multiple="1" display="no" altdistance="0.01" altunitdist="inch" altunit="inch"/>
+<grid distance="0.1" unitdist="inch" unit="inch" style="dots" multiple="1" display="yes" altdistance="0.01" altunitdist="inch" altunit="inch"/>
 <layers>
 <layer number="1" name="Top" color="4" fill="1" visible="no" active="no"/>
@@
 <text x="73.66" y="35.56" size="1.27" layer="94">30V regulated
 output</text>
+<text x="45.72" y="15.24" size="0.8128" layer="94">https://github.com/pksato/TL431-Circuits</text>
 </plain>
 <instances>
